File: speedo-pcb/speedo-pcb.kicad_pcb (KiCad board)
At the start: 4 copper layers, 52 x 52 mm, 66 parts, among them J1 Debug, J2 Mode, J3 Speedo, J4 Power, J5 VBAT, J6 BOOT, J7 Breakout, M1 X27_128, U1 XC6206P332MR, U3 OLED_128x32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

Commit message: pcb clean up
Parts:
- moved C14 2.06 mm to (97.5, 80.7)
- moved C18 2.06 mm to (95.0, 80.7)
- moved X2 2.06 mm to (96.3, 82.2)
- moved C10 1.25 mm to (105.2, 79.8)
- moved C9 1.25 mm to (100.0, 80.5)
- moved X3 1.25 mm to (102.6, 80.1)
Routing:
- net Net-(U4-PC15): track 9.13 -> 6.89 mm
- net Net-(U4-PC14): track 9.95 -> 7.72 mm
- net Net-(U4-PD0): track 10.2 -> 8.97 mm
- net Net-(U4-PD1): track 11.3 -> 10.2 mm
Changed lines of the file:
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@@
 	(footprint "PCM_JLCPCB:C_0402"
 		(layer "B.Cu")
-		(at 96.75 78.75)
+		(at 97.55 80.65)
 		(descr "Capacitor SMD 0402 (1005 Metric), square (rectangular) end terminal, IPC_7351 nominal, (Body size source: IPC-SM-782 page 76, https://www.pcb-3d.com/wordpress/wp-content/uploads/ipc-sm-782a_amendment_1_and_2.pdf), generated with kicad-footprint-generator")
 		(tags "capacitor")
@@
 	(footprint "PCM_JLCPCB:C_0402"
 		(layer "B.Cu")
-		(at 105.25 78.5 -90)
+		(at 105.25 79.75 -90)
 		(descr "Capacitor SMD 0402 (1005 Metric), square (rectangular) end terminal, IPC_7351 nominal, (Body size source: IPC-SM-782 page 76, https://www.pcb-3d.com/wordpress/wp-content/uploads/ipc-sm-782a_amendment_1_and_2.pdf), generated with kicad-footprint-generator")
 		(tags "capacitor")
 		(property "Reference" "C10"
-			(at 1.25 0.75 0)
+			(at 0.05 -0.45 0)
 			(layer "B.SilkS")
 			(effects
@@
 	(footprint "PCM_JLCPCB:C_0402"
 		(layer "B.Cu")
-		(at 94.25 78.75 180)
+		(at 95.05 80.65 180)
 		(descr "Capacitor SMD 0402 (1005 Metric), square (rectangular) end terminal, IPC_7351 nominal, (Body size source: IPC-SM-782 page 76, https://www.pcb-3d.com/wordpress/wp-content/uploads/ipc-sm-782a_amendment_1_and_2.pdf), generated with kicad-footprint-generator")
 		(tags "capacitor")
@@
 	(footprint "PCM_JLCPCB:FC-135R_L3.2-W1.5"
 		(layer "B.Cu")
-		(at 95.5 80.25 180)
+		(at 96.3 82.15 180)
 		(descr "FC-135R_L3.2-W1.5 footprint")
 		(tags "FC-135R_L3.2-W1.5 footprint C32346")
@@
 	(footprint "PCM_JLCPCB:C_0402"
 		(layer "B.Cu")
-		(at 100 79.25 90)
+		(at 100 80.5 90)
 		(descr "Capacitor SMD 0402 (1005 Metric), square (rectangular) end terminal, IPC_7351 nominal, (Body size source: IPC-SM-782 page 76, https://www.pcb-3d.com/wordpress/wp-content/uploads/ipc-sm-782a_amendment_1_and_2.pdf), generated with kicad-footprint-generator")
 		(tags "capacitor")
 		(property "Reference" "C9"
-			(at 1 0.5 0)
+			(at 1.1 0.4 0)
 			(layer "B.SilkS")
 			(effects
@@
 	(footprint "PCM_JLCPCB:OSC-SMD_4P-L3.2-W2.5-BL"
 		(layer "B.Cu")
-		(at 102.6 78.87)
+		(at 102.6 80.12)
 		(descr "OSC-SMD_4P-L3.2-W2.5-BL footprint")
 		(tags "OSC-SMD_4P-L3.2-W2.5-BL footprint C9006")
 		(property "Reference" "X3"
-			(at 0 1.73 0)
+			(at 0 -2.82 0)
 			(layer "B.SilkS")
 			(effects
@@
 			(polygon
 				(pts
-					(xy 100.6 80.47) (xy 104.6 80.47) (xy 104.6 77.27) (xy 100.6 77.27)
+					(xy 100.6 81.72) (xy 104.6 81.72) (xy 104.6 78.52) (xy 100.6 78.52)
 				)
 			)
@@
 	)
 	(via
-		(at 100 80.5)
+		(at 100 81.75)
 		(size 0.6)
 		(drill 0.3)
@@
 	)
 	(via
-		(at 95.5 78.75)
+		(at 96.3 80.65)
 		(size 0.6)
 		(drill 0.3)
@@
 	)
 	(via
-		(at 106 78)
+		(at 106 79.25)
 		(size 0.6)
 		(drill 0.3)
@@
 	)
 	(segment
-		(start 94.75 78.75)
-		(end 95.5 78.75)
+		(start 95.55 80.65)
+		(end 96.3 80.65)
 		(width 0.3)
 		(layer "B.Cu")
@@
 	)
 	(segment
-		(start 101.5 79.75)
-		(end 100 79.75)
+		(start 101.5 81)
+		(end 100 81)
 		(width 0.4)
 		(layer "B.Cu")
@@
 	)
 	(segment
-		(start 101.94 79.75)
-		(end 103.7 77.99)
+		(start 101.94 81)
+		(end 103.7 79.24)
 		(width 0.4)
 		(layer "B.Cu")
@@
 	)
 	(segment
-		(start 100 79.75)
-		(end 100 80.5)
+		(start 100 81)
+		(end 100 81.75)
 		(width 0.4)
 		(layer "B.Cu")
@@
 	)
 	(segment
-		(start 105.25 78)
-		(end 103.71 78)
+		(start 105.25 79.25)
+		(end 103.71 79.25)
 		(width 0.4)
 		(layer "B.Cu")
@@
 	)
 	(segment
-		(start 96.25 78.75)
-		(end 95.5 78.75)
+		(start 97.05 80.65)
+		(end 96.3 80.65)
 		(width 0.3)
 		(layer "B.Cu")
@@
 	)
 	(segment
-		(start 101.5 79.75)
-		(end 101.94 79.75)
+		(start 101.5 81)
+		(end 101.94 81)
 		(width 0.4)
 		(layer "B.Cu")
@@
 	)
 	(segment
-		(start 103.71 78)
-		(end 103.7 77.99)
+		(start 103.71 79.25)
+		(end 103.7 79.24)
 		(width 0.4)
 		(layer "B.Cu")
@@
 	)
 	(segment
-		(start 105.25 78)
-		(end 106 78)
+		(start 105.25 79.25)
+		(end 106 79.25)
 		(width 0.4)
 		(layer "B.Cu")
@@
 	)
 	(segment
-		(start 99.993154 78.75)
-		(end 100 78.75)
+		(start 100.74 80)
+		(end 101.5 79.24)
 		(width 0.3)
 		(layer "B.Cu")
@@
 	)
 	(segment
-		(start 100.74 78.75)
-		(end 101.5 77.99)
+		(start 100 80)
+		(end 100.74 80)
 		(width 0.3)
 		(layer "B.Cu")
@@
 	)
 	(segment
-		(start 100 78.75)
-		(end 100.74 78.75)
+		(start 99.993154 80)
+		(end 100 80)
 		(width 0.3)
 		(layer "B.Cu")
@@
 	)
 	(segment
-		(start 99.25 79.493154)
-		(end 99.993154 78.75)
+		(start 99.25 80.743154)
+		(end 99.993154 80)
 		(width 0.3)
 		(layer "B.Cu")
@@
 	(segment
 		(start 99.25 86.84)
-		(end 99.25 79.493154)
+		(end 99.25 80.743154)
 		(width 0.3)
 		(layer "B.Cu")
@@
 	)
 	(segment
-		(start 103.7 79.75)
-		(end 102.45 81)
+		(start 102.7 82)
+		(end 103.7 81)
 		(width 0.3)
 		(layer "B.Cu")
@@
 	)
 	(segment
-		(start 101.25 81)
-		(end 99.75 82.5)
+		(start 99.75 86.84)
+		(end 99.75 83.493154)
 		(width 0.3)
 		(layer "B.Cu")
@@
 	)
 	(segment
-		(start 99.75 82.5)
-		(end 99.75 86.84)
+		(start 101.243154 82)
+		(end 102.7 82)
 		(width 0.3)
 		(layer "B.Cu")
@@
 	)
 	(segment
-		(start 102.45 81)
-		(end 101.25 81)
+		(start 105.25 80.25)
+		(end 104.45 80.25)
 		(width 0.3)
 		(layer "B.Cu")
@@
 	)
 	(segment
-		(start 105.25 79)
-		(end 104.45 79)
+		(start 104.45 80.25)
+		(end 103.7 81)
 		(width 0.3)
 		(layer "B.Cu")
@@
 	)
 	(segment
-		(start 104.45 79)
-		(end 103.7 79.75)
+		(start 99.75 83.493154)
+		(end 101.243154 82)
 		(width 0.3)
 		(layer "B.Cu")
@@
 	)
 	(segment
-		(start 97.25 78.75)
-		(end 97.25 79.75)
+		(start 98.05 80.65)
+		(end 98.05 81.65)
 		(width 0.3)
 		(layer "B.Cu")
@@
 	)
 	(segment
-		(start 97.25 79.75)
-		(end 96.75 80.25)
+		(start 98.05 81.65)
+		(end 97.55 82.15)
 		(width 0.3)
 		(layer "B.Cu")
@@
 	)
 	(segment
-		(start 98.75 84.25)
-		(end 98.75 86.84)
+		(start 97.55 82.15)
+		(end 98.75 83.35)
 		(width 0.3)
 		(layer "B.Cu")
@@
 	)
 	(segment
-		(start 96.75 80.25)
-		(end 98.75 82.25)
-		(width 0.3)
-		(layer "B.Cu")
-		(net 32)
-	)
-	(segment
-		(start 98.75 82.25)
-		(end 98.75 84.25)
+		(start 98.75 83.35)
+		(end 98.75 86.84)
 		(width 0.3)
 		(layer "B.Cu")
@@
 	)
 	(segment
-		(start 94.25 80.25)
-		(end 98.25 84.25)
+		(start 98.25 85.35)
+		(end 98.25 86.84)
 		(width 0.3)
 		(layer "B.Cu")
@@
 	)
 	(segment
-		(start 98.25 84.25)
-		(end 98.25 86.84)
+		(start 95.05 82.15)
+		(end 98.25 85.35)
 		(width 0.3)
 		(layer "B.Cu")
@@
 	)
 	(segment
-		(start 93.75 79.75)
-		(end 94.25 80.25)
+		(start 94.55 81.65)
+		(end 95.05 82.15)
 		(width 0.3)
 		(layer "B.Cu")
@@
 	)
 	(segment
-		(start 93.75 78.75)
-		(end 93.75 79.75)
+		(start 94.55 80.65)
+		(end 94.55 81.65)
 		(width 0.3)
 		(layer "B.Cu")
